File: powerBoard.sch (KiCad schematic (older format))
At the start: 8 parts, among them U1 ResettableFuse

Commit message: Pushing updates from laptop
Parts:
- removed C1, C2: ELE-101ELL2R2ME11D, SamacSys_Parts:CAPPRD200W50D525H1250, symbol SamacSys_Parts:ELE-101ELL2R2ME11D
- removed U1: ResettableFuse, powerBoardComp:ResettableFuse, symbol powerBoardComp:ResettableFuse
- added C1: 470u, Capacitor_SMD:CP_Elec_18x17.5, symbol Device:CP
- added C10, C11, C8, C9: 1000p, symbol Device:C
- added C12: 3300p, symbol Device:C
- added C13: C, symbol Device:C
- added C2, C4, C5: 470u, SamacSys_Parts:CAPPRD200W50D525H1250, symbol Device:CP
- added C3, C6, C7: 4.7u, Capacitor_SMD:C_1812_4532Metric_Pad1.57x3.40mm_HandSolder, symbol Device:C
- added F1: Polyfuse, powerBoardComp:ResettableFuse, symbol Device:Polyfuse
- added FL1: EMI_Filter_LL_1423, symbol Device:EMI_Filter_LL_1423
- J1: renamed from Vin1; value Screw_Terminal_01x02 -> Vin
- J2: renamed from Vout1; value Screw_Terminal_01x02 -> Vout
- PS1: symbol SamacSys_Parts:RP240H-2448SRW_N-HC -> powerBoard-rescue:RP240H-2448SRW_N-HC-SamacSys_Parts
- R1: value 348 K -> 348K
Connections:
- net VIN+: now reaches J1.2 (Pin_2)
- net VIN+: now also F1.2; no longer PS1.1 (+VIN)
- net VIN-: now reaches J1.1 (Pin_1)
- net VIN-: now also C1.2, C2.2, C3.2, FL1.1; no longer PS1.4 (-VIN)
- net VOUT-: now reaches J2.2 (Pin_2), PS1.5 (-VOUT)
- net VOUT-: now also PS1.6 (-SENSE), R2.2, C11.1, C12.2
- net TRIM: now reaches PS1.7 (TRIM), R1.2, R2.1
- net VOUT+: now reaches PS1.8 (+SENSE), R1.1
- net VOUT+: now also J2.1 (Pin_1), PS1.9 (+VOUT), C10.1, C13.1
- new net GND: C12.1, C13.2, C8.2, C9.2
- new net VIN+_FILTERED: C10.2, C4.1, C5.1, C6.1, C7.1, FL1.3, PS1.1 (+VIN)
- new net VIN+_FUSED: C1.1, C2.1, C3.1, F1.1, FL1.2
- new net VIN-_FILTERED: C11.2, C4.2, C5.2, C6.2, C7.2, C8.1, C9.1, FL1.4, PS1.4 (-VIN)
- no-connect marks 0 -> 1
Other:
- note added: "Design from the RP240 Datasheet\nEMI Filtering according to \nEN55022/11Class A and EN50121-1"
- moved on the sheet: J1, J2, PS1, R1, R2
